Commit message: gazebo-launch

File: urdf/robot.urdf.xacro (robot description, xacro)
@@ -5,4 +5,9 @@
 <!-- base link -->
 <link name="base_link">
+    <inertial>
+        <origin xyz="0.0 0.0 0.0" rpy="0.0 0.0 0.0"/>
+        <mass value="2"/>
+        <inertia ixx="0.0" ixy="0.0" ixz="0.0" iyy="0.0" iyz="0.0" izz="0.0"/>
+    </inertial>
     <visual>
         <origin xyz="0 0 0" rpy="0 0 0" />
@@ -14,4 +19,10 @@
         </material>
     </visual>
+    <collision>
+        <origin xyz="0.0 0.0 0.0" rpy="0.0 0.0 0.0"/>
+        <geometry>
+            <cylinder radius="0.4" length="0.2"/>
+        </geometry>
+    </collision>
 </link>
 <!-- base joint -->
@@ -23,4 +34,9 @@
 <!-- castor wheel -->
 <link name="castor_link">
+    <inertial>
+            <origin xyz="0.0 0.0 0.0" rpy="0.0 0.0 0.0"/>
+            <mass value="1"/>
+            <inertia ixx="0.0" ixy="0.0" ixz="0.0" iyy="0.0" iyz="0.0" izz="0.0"/>
+    </inertial>
     <visual>
         <origin xyz="0 0 0" rpy="0 0 0" />
@@ -32,4 +48,10 @@
         </material>
     </visual>
+    <collision>
+        <origin xyz="0.0 0.0 0.0" rpy="0.0 0.0 0.0"/>
+        <geometry>
+            <sphere radius="0.0445" />
+        </geometry>
+    </collision>
 </link>
 <!-- castor joint  -->
@@ -44,4 +66,9 @@
     <!--wheel link -->
     <link name="wheel_${name}_link">
+        <inertial>
+            <origin xyz="0.0 0.0 0.0" rpy="0.0 0.0 0.0"/>
+            <mass value="1"/>
+            <inertia ixx="0.0" ixy="0.0" ixz="0.0" iyy="0.0" iyz="0.0" izz="0.0"/>
+        </inertial>
         <visual>
             <origin xyz="0 0 0" rpy="0 0 0" />
@@ -53,4 +80,10 @@
             </material>
         </visual>
+        <collision>
+            <origin xyz="0.0 0.0 0.0" rpy="0.0 0.0 0.0"/>
+            <geometry>
+                <mesh filename="package://robot-world/meshes/wheel.stl" scale="0.0034 0.0034 0.0034"/>
+            </geometry>
+        </collision>
     </link>
     <!-- wheel joint  -->
